File: PCB/GrBLDC.kicad_pcb (KiCad board)
At the start: 6 copper layers, 103.1 x 59.6 mm, 209 parts, among them IC1 ATMEGA16M1-A, J1 Conn_02x03_Odd_Even, J2 4910SCK, J3 4910SDI, J4 4910SDO, J5 4910STR, J6 Conn_02x02_Top_Bottom, P1 CONN_6, P10 CONN_8, P11 CONN_2, P12 CONN_01X03, P14 CONN_01X03, P15 CONN_01X03, P2 CONN_8, P3 CONN_01X04, P4 CONN_01X03, P5 CONN_01X05, P6 CONN_01X04, P7 CONN_01X04, P8 CONN_9, P9 CONN_8, Q1 IRF5406, Q2 IRF5406, Q3 IRF5406, Q4 IRF5406, Q5 IRF5406, Q6 IRF5406, U1 DRV8818, U2 DRV8818, U3 DRV8818, U4 DRV8818, U5 A4910, Y1 16M

Commit message: Changed opamp gain offset
opamp offset functionality (i.e. 0A = 8- mV) made gain non-uniform.  Removed opamp offset entirely, as we don't really need it, and I'd rather integrate current more linearly.
Parts:
- R24, R28, R66: value 56k -> DNP
- R68, R70, R72: value 1k -> 47
Changed lines of the file:
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@@
       (effects (font (size 0.75 0.75) (thickness 0.15)))
     )
-    (fp_text value 56k (at 0 1.5 90) (layer F.Fab)
+    (fp_text value DNP (at 0 1.5 90) (layer F.Fab)
       (effects (font (size 1 1) (thickness 0.15)))
     )
@@
       (effects (font (size 0.75 0.75) (thickness 0.15)))
     )
-    (fp_text value 56k (at 0 1.5 270) (layer F.Fab)
+    (fp_text value DNP (at 0 1.5 270) (layer F.Fab)
       (effects (font (size 1 1) (thickness 0.15)))
     )
@@
       (effects (font (size 0.75 0.75) (thickness 0.15)))
     )
-    (fp_text value 1k (at 0 1.5 270) (layer F.Fab)
+    (fp_text value 47 (at 0 1.5 270) (layer F.Fab)
       (effects (font (size 1 1) (thickness 0.15)))
     )
@@
       (effects (font (size 0.75 0.75) (thickness 0.15)))
     )
-    (fp_text value 1k (at 0 1.5 270) (layer F.Fab)
+    (fp_text value 47 (at 0 1.5 270) (layer F.Fab)
       (effects (font (size 1 1) (thickness 0.15)))
     )
@@
       (effects (font (size 0.75 0.75) (thickness 0.15)))
     )
-    (fp_text value 1k (at 0 1.5) (layer F.Fab)
+    (fp_text value 47 (at 0 1.5) (layer F.Fab)
       (effects (font (size 1 1) (thickness 0.15)))
     )
@@
       (effects (font (size 0.75 0.75) (thickness 0.15)))
     )
-    (fp_text value 56k (at 0 1.5 90) (layer F.Fab)
-      (effects (font (size 1 1) (thickness 0.15)))
-    )
+    (fp_text value DNP (at 0 1.5 90) (layer F.Fab)
+      (effects (font (size 1 1) (thickness 0.15)))
+    )
