File: PCB/GrBLDC.sch (KiCad schematic (older format))
At the start: 207 parts, among them IC1 ATMEGA16M1-A, J1 Conn_02x03_Odd_Even, J2 4910SCK, J3 4910SDI, J4 4910SDO, J5 4910STR, J6 Conn_02x02_Top_Bottom, P1 CONN_6, P10 CONN_8, P11 CONN_2, P12 CONN_01X03, P14 CONN_01X03, P15 CONN_01X03, P2 CONN_8, P3 CONN_01X04, P4 CONN_01X03, P5 CONN_01X05, P6 CONN_01X04, P7 CONN_01X04, P8 CONN_9, P9 CONN_8, Q1 IRF5406, Q2 IRF5406, Q3 IRF5406, Q4 IRF5406, Q5 IRF5406, Q6 IRF5406, U1 DRV8818, U2 DRV8818, U3 DRV8818, U4 DRV8818, U5 A4910, Y1 16M

Commit message: Changed opamp gain offset
opamp offset functionality (i.e. 0A = 8- mV) made gain non-uniform.  Removed opamp offset entirely, as we don't really need it, and I'd rather integrate current more linearly.
Parts:
- R24, R28, R66: value 56k -> DNP
- R68, R70, R72: value 1k -> 47
